Commit message: Add finger gripper to UR robots
Signed-off-by: Artur Kamieniecki <artur.kamieniecki@robotec.ai>
Signed-off-by: Jan Hanca <jan.hanca@robotec.ai>

File: ros2_ws/src/Universal_Robots_ROS2_Description/urdf/finger_gripper/hand.xacro (robot description, xacro)
@@ -12,10 +12,10 @@
       <visual>
         <geometry>
-          <mesh filename="package://franka_description/meshes/robot_ee/franka_hand_white/visual/hand.dae"/>
+          <mesh filename="package://ur_description/meshes/finger_gripper/visual/hand.dae"/>
         </geometry>
       </visual>
       <collision>
         <geometry>
-          <mesh filename="package://franka_description/meshes/robot_ee/franka_hand_white/collision/hand.stl"/>
+          <mesh filename="package://ur_description/meshes/finger_gripper/collision/hand.stl"/>
         </geometry>
       </collision>
@@ -29,10 +29,10 @@
       <visual>
         <geometry>
-          <mesh filename="package://franka_description/meshes/robot_ee/franka_hand_white/visual/finger.dae"/>
+          <mesh filename="package://ur_description/meshes/finger_gripper/visual/finger.dae"/>
         </geometry>
       </visual>
       <collision>
         <geometry>
-          <mesh filename="package://franka_description/meshes/robot_ee/franka_hand_white/collision/finger.stl"/>
+          <mesh filename="package://ur_description/meshes/finger_gripper/collision/finger.stl"/>
         </geometry>
       </collision>
@@ -47,5 +47,5 @@
         <origin xyz="0 0 0" rpy="0 0 ${pi}"/>
         <geometry>
-          <mesh filename="package://franka_description/meshes/robot_ee/franka_hand_white/visual/finger.dae"/>
+          <mesh filename="package://ur_description/meshes/finger_gripper/visual/finger.dae"/>
         </geometry>
       </visual>
@@ -53,5 +53,5 @@
         <origin xyz="0 0 0" rpy="0 0 ${pi}"/>
         <geometry>
-          <mesh filename="package://franka_description/meshes/robot_ee/franka_hand_white/collision/finger.stl"/>
+          <mesh filename="package://ur_description/meshes/finger_gripper/collision/finger.stl"/>
         </geometry>
       </collision>

File: ros2_ws/src/Universal_Robots_ROS2_Description/urdf/ur_macro.xacro (robot description, xacro)
@@ -44,4 +44,5 @@
   <xacro:include filename="$(find ur_description)/urdf/inc/ur_transmissions.xacro" />
   <xacro:include filename="$(find ur_description)/urdf/inc/ur_common.xacro" />
+  <xacro:include filename="$(find ur_description)/urdf/finger_gripper/hand.xacro" />
   <xacro:macro name="ur_robot" params="
     name
@@ -252,18 +253,4 @@
       </xacro:cylinder_inertial>
     </link>
-    <link name="${tf_prefix}gripper_link">
-      <visual>
-        <origin xyz="0 0 0" rpy="${pi/2} 0 ${-pi/2}"/>
-        <geometry>
-          <xacro:get_mesh name="gripper" type="visual"/>
-        </geometry>
-      </visual>
-      <collision>
-        <origin xyz="0 0 0" rpy="${pi/2} 0 ${-pi/2}"/>
-        <geometry>
-          <xacro:get_mesh name="gripper" type="collision"/>
-        </geometry>
-      </collision>
-    </link>
     <!-- base_joint fixes base_link to the environment -->
     <joint name="${tf_prefix}base_joint" type="fixed">
@@ -388,9 +375,6 @@
       <child link="${tf_prefix}tool0"/>
     </joint>
-    <joint name="${tf_prefix}tool0-gripper" type="fixed">
-      <origin xyz="0 0 0.10" rpy="${pi/2.0} ${pi/2.0} 0"/>
-      <parent link="${tf_prefix}tool0"/>
-      <child link="${tf_prefix}gripper_link"/>
-    </joint>
+    <!-- Attach Panda hand under tool0 -->
+    <xacro:hand connected_to="${tf_prefix}tool0" ns="${tf_prefix}panda" rpy="0 0 0" xyz="0 0 0"/>
   </xacro:macro>
 </robot>
