Commit message: Modify UR driver
Signed-off-by: Artur Kamieniecki <artur.kamieniecki@robotec.ai>

File: ros2_ws/src/Universal_Robots_ROS2_Driver/ur_moveit_config/srdf/ur_macro.srdf.xacro (robot description, xacro)
@@ -13,4 +13,9 @@
     <group name="${prefix}${name}_manipulator">
       <chain base_link="${prefix}base_link" tip_link="${prefix}tool0" />
+    </group>
+    <!-- Panda gripper planning group -->
+    <group name="${prefix}${name}_gripper">
+      <joint name="${prefix}panda_finger_joint1"/>
+      <joint name="${prefix}panda_finger_joint2"/>
     </group>
     <!--GROUP STATES - Purpose - Define a named state for a particular group, in terms of joint values. This is useful to define states like 'folded arms'-->
@@ -39,4 +44,13 @@
       <joint name="${prefix}wrist_3_joint" value="-0.11" />
     </group_state>
+    <!-- Gripper group states -->
+    <group_state name="${prefix}open" group="${prefix}${name}_gripper">
+      <joint name="${prefix}panda_finger_joint1" value="0.04"/>
+      <joint name="${prefix}panda_finger_joint2" value="0.04"/>
+    </group_state>
+    <group_state name="${prefix}closed" group="${prefix}${name}_gripper">
+      <joint name="${prefix}panda_finger_joint1" value="0.0"/>
+      <joint name="${prefix}panda_finger_joint2" value="0.0"/>
+    </group_state>
     <!--END EFFECTOR - Purpose - Represent information about an end effector.-->
     <!--VIRTUAL JOINT - Purpose - this element defines a virtual joint between a robot link and an external frame of reference (considered fixed with respect to the robot)-->
@@ -53,4 +67,10 @@
     <disable_collisions link1="${prefix}wrist_1_link" link2="${prefix}wrist_3_link" reason="Never" />
     <disable_collisions link1="${prefix}wrist_2_link" link2="${prefix}wrist_3_link" reason="Adjacent" />
+    <!-- Disable collisions for Panda hand -->
+    <disable_collisions link1="${prefix}wrist_3_link" link2="${prefix}panda_hand" reason="Adjacent" />
+    <disable_collisions link1="${prefix}tool0" link2="${prefix}panda_hand" reason="Adjacent" />
+    <disable_collisions link1="${prefix}panda_hand" link2="${prefix}panda_leftfinger" reason="Adjacent" />
+    <disable_collisions link1="${prefix}panda_hand" link2="${prefix}panda_rightfinger" reason="Adjacent" />
+    <disable_collisions link1="${prefix}panda_leftfinger" link2="${prefix}panda_rightfinger" reason="Default" />
   </xacro:macro>
 </robot>
